File: PiKey_KiCad/PiKey_KiCad.kicad_pcb (KiCad board)
At the start: 4 copper layers, 22 x 42 mm, 25 parts, among them J1 SWD Header, SW1 BOOTSEL, SW2 RESET, U1 W25Q32JVSS, U2 RP2040, Y1 Crystal

Commit message: Fixed page settings, added BOM
Changed lines of the file:
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@@
   )
   (paper "A4")
+  (title_block
+    (title "PiKey: RP2040 M.2 B+M SoM")
+    (date "2023-09-15")
+    (rev "v1.0")
+  )
   (layers
     (0 "F.Cu" signal)
@@
   (gr_circle (center 149.3 104.8) (end 149.441421 104.8)
     (stroke (width 0.15) (type solid)) (fill solid) (layer "F.SilkS"))
-  (gr_circle (center 152.55 113.25) (end 152.691421 113.25)
+  (gr_circle (center 153.65 113.25) (end 153.791421 113.25)
     (stroke (width 0.15) (type solid)) (fill solid) (layer "F.SilkS"))
   (gr_circle (center 140.85 97.45) (end 140.991421 97.45)
@@
     (pts (xy 164.4 86.7) (xy 164.4 128.7))
     (height 0)
-    (gr_text "1653.5433 mils" (at 163.25 107.7 90) (layer "Dwgs.User")
+    (gr_text "42.0000 mm" (at 163.25 107.7 90) (layer "Dwgs.User")
       (effects (font (size 1 1) (thickness 0.15)))
     )
@@
     (pts (xy 138.4 82.7) (xy 160.4 82.7))
     (height 0)
-    (gr_text "866.1417 mils" (at 149.4 81.55) (layer "Dwgs.User")
+    (gr_text "22.0000 mm" (at 149.4 81.55) (layer "Dwgs.User")
       (effects (font (size 1 1) (thickness 0.15)))
     )
